File: project/ZSWatch-Dock.kicad_pcb (KiCad board)
At the start: 2 copper layers, 52 x 52 mm, 37 parts, among them IC1 XC9265C181MR-G, IC2 MIC5219-3.3YM5, IC3 NTS0104GU12, IC4 STM32F072CBT6, SW1 CONFIG, X1 WATCH, X2 GPIO, X3 DEBUG, X4 USB4105-GF-A

Commit message: - Add missing 3D model for IC1 - Adjust silkscreen on the botton - Add right footprint for debug connector - Generate new production data - Add BOM variants for option with and without J-Link - Add missing part numbers for R4 to R6 - Add missing part numbers for R1 to R3 - Add BOM for PCBWay - Update page template to newest KiCad version - Update step file - Replace DIP switch - Add specification for Segger OB Debugger - Swap RxD and TxD of the STM32 to align it with the Segger OB Debugger specification
Signed-off-by: Daniel Kampert <DanielKampert@kampis-elektroecke.de>
Parts:
- X3: footprint Connector_PinHeader_1.27mm:PinHeader_2x05_P1.27mm_Vertical_SMD -> Samtec:SHF-105-01-L-D-SM-TR
- moved G*** 12.8 mm to (156.5, 120.5)
- moved G*** 11.7 mm to (149.0, 120.0)
Connections:
- IC4 pad 29: GPIO -> unconnected-(IC4-PA8-Pad29)
- IC4 pad 30: STM32_RxD -> STM32_TxD
- IC4 pad 31: STM32_TxD -> STM32_RxD
Routing:
- net GPIO: track 20.3 -> 9.35 mm
- net STM32_TxD: track 23.6 -> 19.3 mm
- net STM32_RxD: track 18.4 -> 19.1 mm
- net GND: track 31.3 -> 30.7 mm

Commit message: - Reorganize the production files and prepare everything for an easy ordering at PCBWay - Replace schematic symbol for debug connector with standard KiCad part - Enable print part value option in Gerber to fix missing documentation on the PCB - Update README
Signed-off-by: Daniel Kampert <DanielKampert@kampis-elektroecke.de>
Parts:
- renumbered R4 to R1, R5 to R2, R6 to R3

Commit message: - Sync designators in BOM with Schematics - Update all production files for the configuration with J-Link
Parts:
- removed the R1 at (155.1, 102.8)
- removed the R2 at (155.1, 101.3)
- removed the R3 at (151.8, 101.4)
- added R4: 0R, Resistor_SMD:R_0603_1608Metric, F.Cu at (155.0, 102.8)
- added R5: 0R, Resistor_SMD:R_0603_1608Metric, F.Cu at (155.0, 101.3)
- added R6: 0R, Resistor_SMD:R_0603_1608Metric, F.Cu at (151.7, 101.4)
- R7, R8: value 5.1k -> 5k1

Commit message: - Add signal names on silkscreen for watch connector - Add production data for variant without J-Link
Parts:
- moved G*** 6.07 mm to (138.1, 90.2)
Other:
- board text added: "GND"
- board text added: "SWDCLK"
- board text added: "SWDIO"
- board text added: "VBUS"
- board text added: "~{Reset}"
Changed lines of the file:
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@@
     (property "ki_description" "Resistor, small symbol")
     (property "ki_keywords" "R resistor")
-    (attr smd exclude_from_bom)
+    (attr smd exclude_from_pos_files exclude_from_bom)
     (fp_text reference "R6" (at 0 -1.43 90) (layer "F.SilkS") hide
         (effects (font (size 1 1) (thickness 0.15)))
@@
         (effects (font (size 0.8 0.8) (thickness 0.12)))
     )
-    (fp_text user "${REFERENCE}" (at 0.0015 -2.459 180) (layer "F.Fab")
+    (fp_text user "${REFERENCE}" (at 0.0015 5.053 180) (layer "F.Fab")
         (effects (font (size 1 1) (thickness 0.15)))
     )
@@
         (effects (font (size 1 1) (thickness 0.15)))
     )
-    (fp_text user "${REFERENCE}" (at 0 0) (layer "F.Fab")
+    (fp_text user "${REFERENCE}" (at 0 -1.142) (layer "F.Fab")
         (effects (font (size 1 1) (thickness 0.15)))
     )
@@
     (property "ki_description" "Resistor, small symbol")
     (property "ki_keywords" "R resistor")
-    (attr smd exclude_from_bom)
+    (attr smd exclude_from_pos_files exclude_from_bom)
     (fp_text reference "R4" (at 0 -1.43) (layer "F.SilkS") hide
         (effects (font (size 1 1) (thickness 0.15)))
@@
   )
   (footprint "LOGO" (layer "F.Cu")
-    (at 141.986 94.869)
+    (at 138.1 90.2)
     (attr board_only exclude_from_pos_files exclude_from_bom)
     (fp_text reference "G***" (at 0 -5.08) (layer "User.1") hide
@@
     (property "ki_description" "Resistor, small symbol")
     (property "ki_keywords" "R resistor")
-    (attr smd exclude_from_bom)
+    (attr smd exclude_from_pos_files exclude_from_bom)
     (fp_text reference "R5" (at 0 -1.43) (layer "F.SilkS") hide
         (effects (font (size 1 1) (thickness 0.15)))
@@
       (stroke (width 0) (type solid)) (fill solid) (layer "B.SilkS"))
   )
+  (gr_line (start 144.388 84.593) (end 164.2 84.593)
+    (stroke (width 0.1) (type default)) (layer "F.SilkS"))
   (gr_circle (center 158.115 77.978) (end 158.315 77.978)
     (stroke (width 0.4) (type default)) (fill none) (layer "F.SilkS"))
+  (gr_line (start 164.2 89.8) (end 144.388 89.8)
+    (stroke (width 0.1) (type default)) (layer "F.SilkS"))
+  (gr_line (start 144.388 89.8) (end 144.388 84.593)
+    (stroke (width 0.1) (type default)) (layer "F.SilkS"))
+  (gr_line (start 164.2 84.593) (end 164.2 89.8)
+    (stroke (width 0.1) (type default)) (layer "F.SilkS"))
   (gr_circle (center 154.1765 100.249) (end 180.1765 100.249)
     (stroke (width 0.254) (type solid)) (fill none) (layer "Edge.Cuts"))
@@
   (gr_line (start 116.455573 12.827) (end 116.455573 45.827)
     (stroke (width 0.1) (type default)) (layer "User.1"))
-  (gr_line (start 134.9995 84.501) (end 154.8115 84.501)
-    (stroke (width 0.1) (type default)) (layer "User.1"))
   (gr_line (start 72.177 12.827) (end 72.177 45.827)
     (stroke (width 0.1) (type default)) (layer "User.1"))
@@
   (gr_line (start 12.827 45.827) (end 133.04843 45.827)
     (stroke (width 0.1) (type default)) (layer "User.1"))
-  (gr_line (start 154.8115 89.708) (end 134.9995 89.708)
-    (stroke (width 0.1) (type default)) (layer "User.1"))
   (gr_line (start 133.04843 12.827) (end 133.04843 45.827)
     (stroke (width 0.1) (type default)) (layer "User.1"))
   (gr_line (start 12.827 12.827) (end 133.04843 12.827)
     (stroke (width 0.1) (type default)) (layer "User.1"))
-  (gr_line (start 134.9995 89.708) (end 134.9995 84.501)
-    (stroke (width 0.1) (type default)) (layer "User.1"))
   (gr_line (start 103.719858 12.827) (end 103.719858 45.827)
     (stroke (width 0.1) (type default)) (layer "User.1"))
@@
   (gr_line (start 12.827 16.577) (end 133.04843 16.577)
     (stroke (width 0.1) (type default)) (layer "User.1"))
-  (gr_line (start 154.8115 84.501) (end 154.8115 89.708)
-    (stroke (width 0.1) (type default)) (layer "User.1"))
   (gr_line (start 12.827 12.827) (end 12.827 45.827)
     (stroke (width 0.1) (type default)) (layer "User.1"))
@@
     (effects (font (size 0.8 0.8) (thickness 0.12)) (justify right mirror))
   )
+  (gr_text "~{Reset}" (at 135.7 102.5) (layer "F.SilkS")
+    (effects (font (size 0.8 0.8) (thickness 0.12)) (justify left bottom))
+  )
   (gr_text "RxD" (at 155.5735 123.109 90) (layer "F.SilkS")
     (effects (font (size 0.8 0.8) (thickness 0.12)) (justify left bottom))
@@
     (effects (font (size 0.8 0.8) (thickness 0.12)) (justify left bottom))
   )
+  (gr_text "VBUS" (at 135.4 107.6) (layer "F.SilkS")
+    (effects (font (size 0.8 0.8) (thickness 0.12)) (justify left bottom))
+  )
+  (gr_text "SWDCLK" (at 135.7 97.3) (layer "F.SilkS")
+    (effects (font (size 0.8 0.8) (thickness 0.12)) (justify left bottom))
+  )
+  (gr_text "Important:\nFor use with ZSWatch only.\nSEGGER OB Licence Required" (at 145.023 87.26) (layer "F.SilkS")
+    (effects (font (size 0.8 0.8) (thickness 0.12)) (justify left))
+  )
   (gr_text "GPIO" (at 158.2405 122.982 90) (layer "F.SilkS")
     (effects (font (size 0.8 0.8) (thickness 0.12)) (justify left bottom))
   )
+  (gr_text "GND" (at 135.6 105.1) (layer "F.SilkS")
+    (effects (font (size 0.8 0.8) (thickness 0.12)) (justify left bottom))
+  )
   (gr_text "Reset" (at 150.4935 123.109 90) (layer "F.SilkS")
     (effects (font (size 0.8 0.8) (thickness 0.12)) (justify left bottom))
   )
+  (gr_text "SWDIO" (at 135.6 99.9) (layer "F.SilkS")
+    (effects (font (size 0.8 0.8) (thickness 0.12)) (justify left bottom))
+  )
   (gr_text "Metallisierte Platinenkante: " (at 201.642995 31.704) (layer "User.1")
     (effects (font (size 1.5 1.5) (thickness 0.2)) (justify left top))
@@
     (effects (font (size 1.5 1.5) (thickness 0.1)) (justify left top))
   )
-  (gr_text "Important:\nFor use with ZSWatch only.\nSEGGER OB Licence Required" (at 135.6345 87.168) (layer "User.1")
-    (effects (font (size 0.8 0.8) (thickness 0.12)) (justify left))
-  )
   (gr_text "Dielektrikum 1" (at 13.577 30.327) (layer "User.1")

Commit message: - Add blue color to PCB settings - Add surface option to PCB settings
Signed-off-by: Daniel Kampert <DanielKampert@kampis-elektroecke.de>
Other:
- board text added: "52,0000 mm x 52,0000 mm"
- board text added: "HAL lead-free"
- board text removed: "53,6979 mm x 53,7004 mm"
- board text removed: "None"

Commit message: - Streamline documentation and production files - Ready to merge
Other:
- board text added: "FR4 natural"
- board text added: "Green"
- board text added: "HAL SnPb"
- board text added: "White"
- board text removed: "HAL lead-free"

Commit message: Initialize branch, add dip switch to enable / disable charging
Other:
- board text added: "1.0.3"
- board text removed: "1.0.2"
Changed lines of the file:
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@@
     (title "ZSWatch Dock Programmer and Charger")
     (date "2023-09-27")
-    (rev "2")
+    (rev "3")
     (company "github.com/jakkra/ZSWatch-Dock")
   )
@@
   (gr_line (start 13.1 39.5) (end 131.678571 39.5)
     (stroke (width 0.1) (type default)) (layer "User.1"))
-  (gr_text "1.0.2" (at 155.702 124.968) (layer "B.Cu")
+  (gr_text "1.0.3" (at 155.702 124.968) (layer "B.Cu")
     (effects (font (size 0.8 0.8) (thickness 0.12)) (justify left bottom mirror))
   )

Commit message: - Add QR code with link to GitHub repository - Add switch to enable / disable charging - Remove reset line from STM32 to the watch connector
Signed-off-by: Daniel Kampert <DanielKampert@kampis-elektroecke.de>
Parts:
- removed SW1: CONFIG, Button_Switch_SMD:SW_DIP_SPSTx04_Slide_Omron_A6S-410x_W8.9mm_P2.54mm
- removed X2: GPIO, Connector_PinHeader_2.54mm:PinHeader_1x01_P2.54mm_Vertical
- added D3: DEBUG, LED_SMD:LED_0603_1608Metric, F.Cu at (165.8, 121.3)
- added G***: LOGO, project:QR-Code, B.Cu at (153.5, 83.7)
- added Q1: BSH205G2AR, Package_TO_SOT_SMD:SOT-23, F.Cu at (164.1, 111.5)
- added R10: 220R, Resistor_SMD:R_0603_1608Metric, F.Cu at (163.6, 119.1)
- added R9: 100k, Resistor_SMD:R_0603_1608Metric, F.Cu at (166.9, 111.4)
- added SW2: CHARGE, Button_Switch_SMD:SW_SP3T_PCM13, F.Cu at (170.6, 116.4)
- added kibuzzard-6522ABB2: G***, kibuzzard-6522ABB2, F.Cu at (173.5, 90.2)
- added kibuzzard-6522ABCA: G***, kibuzzard-6522ABCA, F.Cu at (173.5, 93.4)
- added kibuzzard-6525026C: G***, kibuzzard-6525026C, F.Cu at (163.2, 121.0)
- moved G*** 22.2 mm to (154.9, 115.7)
- moved C1 11.3 mm to (158.9, 110.1)
- moved C2 11.3 mm to (156.0, 115.1)
- moved IC1 11.3 mm to (158.6, 113.0)
- moved L1 11.3 mm to (158.6, 115.9)
- moved G*** 1.54 mm to (156.9, 122.0)
- moved G*** 1.54 mm to (149.4, 121.5)
Connections:
- IC3 pad 10: /SWDRESETn -> unconnected-(IC3-B1-Pad10)
- IC3 pad 2: STM32_SWD_RESETn -> unconnected-(IC3-A1-Pad2)
- IC4 pad 11: /SWDRESETn -> unconnected-(IC4-PA1-Pad11)
- IC4 pad 30: STM32_TxD -> unconnected-(IC4-PA9-Pad30)
- IC4 pad 31: STM32_RxD -> unconnected-(IC4-PA10-Pad31)
- X1 pad 3: ZSWatch_RESETn -> GND
- X1 pad 5: VBUS -> Net-(Q1-D)
Routing:
- net ZSWatch_RESETn: track 36.6 -> 0.00 mm
- net VBUS: track 35.3 -> 3.23 mm, vias 1 -> 0
- net Net-(Q1-D): track 0.00 -> 31.3 mm, vias 0 -> 1
- net STM32_TxD: track 19.3 -> 0.00 mm, vias 2 -> 0
- net STM32_RxD: track 19.1 -> 0.00 mm, vias 2 -> 0
- net STM32_SWD_RESETn: track 13.1 -> 0.00 mm, vias 2 -> 0
- net unconnected-(IC3-A1-Pad2): track 0.00 -> 11.0 mm, vias 0 -> 2
- net +1V8: track 41.6 -> 31.1 mm, vias 4 -> 3
- net GPIO: track 9.35 -> 0.00 mm
- net Net-(Q1-G): track 0.00 -> 7.20 mm
- net CHARGE: track 0.00 -> 7.02 mm
- net GND: track 30.7 -> 32.9 mm, vias 17 -> 19
- net Net-(D3-K): track 0.00 -> 1.51 mm
- net STATUS: track 37.9 -> 37.3 mm
Other:
- board text added: "Dock and debugger v1 Rev 3"
- board text added: "USB/SWD"
- board text removed: "Dock and debugger v1 Rev 2"
- board text removed: "GPIO"
- board text removed: "Reset"
- board text removed: "RxD"
- board text removed: "TxD"
- board text removed: "~{Reset}"
