File: project/ZSWatch-Dock.kicad_pcb (KiCad board)
At the start: 2 copper layers, 50 x 55 mm, 58 parts, among them IC1 XC9265C181MR-G, IC2 TS3USB221A, IC3 MIC5219-3.3YM5, IC4 NTS0104GU12, IC5 STM32F072CBT6, Q1 BSH205G2AR, SW1 SEL, SW2 CHARGE, X1 WATCH, X2 DEBUG, X3 DEBUG, X4 DATA

Commit message: Add debounce capacitor to SEL-Switch
Parts:
- added C2: 100n, Capacitor_SMD:C_0603_1608Metric, F.Cu at (164.0, 116.0)
- added R3: 1k, Resistor_SMD:R_0603_1608Metric, F.Cu at (151.1, 121.8)
- renumbered C9 to C10, C10 to C11, C11 to C12, C12 to C13, C2 to C3, C3 to C4, C4 to C5, C5 to C6, C6 to C7, C7 to C8, C8 to C9, R9 to R10, R10 to R11, R11 to R12, R12 to R13, R13 to R14, R14 to R15, R15 to R16, R16 to R17, R17 to R18, R3 to R2, R2 to R4, R4 to R5, R5 to R6, R6 to R7, R7 to R8, R8 to R9
Connections:
- SW1 pad 3: SEL_SWD -> Net-(SW1A-C)
Routing:
- net SEL_SWD: track 48.8 -> 45.8 mm
- net Net-(SW1A-C): track 0.00 -> 2.85 mm
- net GND: track 42.2 -> 43.1 mm, vias 24 -> 25

Commit message: Change power supply for CHARGE LED to VBUS
Parts:
- D3: value DEBUG -> CHARGE
Connections:
- D3 pad 2: +3V3 -> VBUS
Routing:
- net VBUS: track 3.23 -> 21.1 mm
Changed lines of the file:
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@@
     (descr "LED SMD 0603 (1608 Metric), square (rectangular) end terminal, IPC_7351 nominal, (Body size source: http://www.tortai-tech.com/upload/download/2011102023233369053.pdf), generated with kicad-footprint-generator")
     (tags "LED")
+    (property "CONFIG" "")
     (property "Distributor" "Mouser")
     (property "Mfr." "Wurth Elektronik")
@@
         (effects (font (size 1 1) (thickness 0.15)))
     )
-    (fp_text value "DEBUG" (at 0 1.43 90) (layer "F.Fab") hide
+    (fp_text value "CHARGE" (at 0 1.43 90) (layer "F.Fab") hide
         (effects (font (size 1 1) (thickness 0.15)))
     )
@@
       (net 61 "Net-(D3-K)") (pinfunction "K") (pintype "passive"))
     (pad "2" smd roundrect (at 0.7875 0 270) (size 0.875 0.95) (layers "F.Cu" "F.Paste" "F.Mask") (roundrect_rratio 0.25)
-      (net 3 "+3V3") (pinfunction "A") (pintype "passive"))
+      (net 9 "VBUS") (pinfunction "A") (pintype "passive"))
     (model "${KICAD6_3DMODEL_DIR}/LED_SMD.3dshapes/LED_0603_1608Metric.wrl"
       (offset (xyz 0 0 0))
@@
   (via (at 154.813 106.553) (size 0.8) (drill 0.4) (layers "F.Cu" "B.Cu") (net 8))
   (segment (start 173.864 104.5465) (end 173.9775 104.433) (width 0.508) (layer "B.Cu") (net 8))
+  (segment (start 161.036 113.945) (end 159.391 112.3) (width 0.4) (layer "F.Cu") (net 9))
   (segment (start 157.766 112.575) (end 159.116 112.575) (width 0.4) (layer "F.Cu") (net 9))
   (segment (start 159.391 112.3) (end 159.391 111.75) (width 0.4) (layer "F.Cu") (net 9))
   (segment (start 159.116 112.575) (end 159.391 112.3) (width 0.4) (layer "F.Cu") (net 9))
+  (segment (start 158.623 126.746) (end 157.607 125.73) (width 0.4) (layer "F.Cu") (net 9))
+  (segment (start 157.607 125.73) (end 157.607 120.269) (width 0.4) (layer "F.Cu") (net 9))
+  (segment (start 159.512 126.746) (end 158.623 126.746) (width 0.4) (layer "F.Cu") (net 9))
   (segment (start 157.491 111.75) (end 157.491 112.3) (width 0.4) (layer "F.Cu") (net 9))
   (segment (start 157.491 112.3) (end 157.766 112.575) (width 0.4) (layer "F.Cu") (net 9))
+  (segment (start 161.036 116.84) (end 161.036 113.945) (width 0.4) (layer "F.Cu") (net 9))
+  (segment (start 157.607 120.269) (end 161.036 116.84) (width 0.4) (layer "F.Cu") (net 9))
   (segment (start 173.72 117.45) (end 174.864 117.45) (width 0.2) (layer "F.Cu") (net 10))
   (segment (start 175.044 117.63) (end 175.044 118.278) (width 0.2) (layer "F.Cu") (net 10))

Commit message: Cosmetic changes
Parts:
- moved C2 1.29 mm to (165.2, 116.0)
- moved R4 1.29 mm to (166.8, 116.0)
- moved R1 0.13 mm to (163.8, 79.9)
- moved R2 0.13 mm to (162.3, 79.9)
- moved C11 0.11 mm to (151.4, 94.6)
Routing:
- net CHARGE: track 24.5 -> 25.9 mm
- net GND: track 43.1 -> 42.2 mm
- net SEL_SWD: vias 3 -> 2

Commit message: Remove color information for soldermask from project
Other:
- board text added: "PCBWay 2-Layer Stack"
- board text added: "Verlustfaktor"
- board text removed: "Green"
- board text removed: "Verlustwinkel"
