File: project/ZSWatch-Dock.kicad_sch (KiCad schematic)
At the start: 31 parts, among them IC1 XC9265C181MR-G, IC2 MIC5219-3.3YM5, IC3 NTS0104GU12, IC4 STM32F072CBT6, SW1 CONFIG, X1 WATCH, X2 GPIO, X3 DEBUG, X4 USB4105-GF-A

Commit message: Initialize branch, add dip switch to enable / disable charging
Parts:
- added SW2: CHARGE, Button_Switch_SMD:SW_DIP_SPSTx01_Slide_6.7x4.1mm_W6.73mm_P2.54mm_LowProfile_JPin, symbol Switch:SW_DIP_x01
- SW1: symbol Switch:SW_DIP_x04 -> Switch:SW_DIP_x01
Connections:
- net GPIO: no longer SW1.5
- net STM32_RxD: now also SW1.2; no longer SW1.6
- net STM32_SWD_RESETn: no longer SW1.8
- net STM32_TxD: no longer SW1.7
- net VBUS: now also SW2.2; no longer X1.5 (Pin_5)
- net ZSWatch_RESETn: no longer SW1.2, SW1.3, SW1.4
- new net: SW2.1, X1.5 (Pin_5)
Changed lines of the file:
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@@
     (title "ZSWatch Dock Programmer and Charger")
     (date "2023-09-27")
-    (rev "2")
+    (rev "3")
     (company "github.com/jakkra/ZSWatch-Dock")
   )
@@
     (stroke (width 0) (type default))
   )
-  (wire (pts (xy 53.34 91.44) (xy 53.34 95.25))
-    (stroke (width 0) (type default))
-  )
   (wire (pts (xy 130.81 66.04) (xy 132.08 66.04))
     (stroke (width 0) (type default))
@@
     (stroke (width 0) (type default))
   )
+  (wire (pts (xy 53.34 97.79) (xy 53.34 99.06))
+    (stroke (width 0) (type default))
+  )
   (wire (pts (xy 110.49 30.48) (xy 120.65 30.48))
     (stroke (width 0) (type default))
@@
     (stroke (width 0) (type dash_dot))
   )
+  (wire (pts (xy 34.29 99.06) (xy 34.29 95.25))
+    (stroke (width 0) (type default))
+  )
   (wire (pts (xy 143.51 41.91) (xy 146.05 41.91))
     (stroke (width 0) (type default))
@@
     (stroke (width 0) (type default))
   )
-  (wire (pts (xy 29.21 95.25) (xy 53.34 95.25))
+  (wire (pts (xy 29.21 95.25) (xy 34.29 95.25))
     (stroke (width 0) (type default))
   )
@@
     (stroke (width 0) (type dash_dot))
   )
+  (wire (pts (xy 52.07 99.06) (xy 53.34 99.06))
+    (stroke (width 0) (type default))
+  )
   (polyline (pts (xy 13.97 167.64) (xy 66.04 167.64))
     (stroke (width 0) (type dash_dot))
@@
   )
   (wire (pts (xy 78.74 26.67) (xy 78.74 30.48))
+    (stroke (width 0) (type default))
+  )
+  (wire (pts (xy 36.83 99.06) (xy 34.29 99.06))
     (stroke (width 0) (type default))
   )
@@
     )
   )
+  (symbol (lib_id "Switch:SW_DIP_x01") (at 44.45 99.06 0) (unit 1)
+    (in_bom yes) (on_board yes) (dnp no) (fields_autoplaced)
+    (property "Reference" "SW2" (at 44.45 92.71 0)
+      (effects (font (size 1.27 1.27)))
+    )
+    (property "Value" "CHARGE" (at 44.45 95.25 0)
+      (effects (font (size 1.27 1.27)))
+    )
+    (property "Footprint" "Button_Switch_SMD:SW_DIP_SPSTx01_Slide_6.7x4.1mm_W6.73mm_P2.54mm_LowProfile_JPin" (at 44.45 99.06 0)
+      (effects (font (size 1.27 1.27)) hide)
+    )
+    (property "Datasheet" "~" (at 44.45 99.06 0)
+      (effects (font (size 1.27 1.27)) hide)
+    )
+    (property "Mfr." "" (at 44.45 99.06 0)
+      (effects (font (size 1.27 1.27)) hide)
+    )
+    (property "Mfr. No." "" (at 44.45 99.06 0)
+      (effects (font (size 1.27 1.27)) hide)
+    )
+    (property "Distributor" "" (at 44.45 99.06 0)
+      (effects (font (size 1.27 1.27)) hide)
+    )
+    (property "Order Number" "" (at 44.45 99.06 0)
+      (effects (font (size 1.27 1.27)) hide)
+    )
+    (pin "1")
+    (pin "2")
+    (instances
+      (project "ZSWatch-Dock"
+        (path "/74a2d9cd-6788-49ca-9d1d-a5e7b3102f3e"
+          (reference "SW2") (unit 1)
+        )
+      )
+    )
+  )
   (symbol (lib_id "Device:L_Small") (at 55.88 29.21 90) (unit 1)
     (in_bom yes) (on_board yes) (dnp no) (fields_autoplaced)
@@
     )
   )
-  (symbol (lib_id "power:VBUS") (at 53.34 91.44 0) (mirror y) (unit 1)
-    (in_bom yes) (on_board yes) (dnp no)
-    (property "Reference" "#PWR08" (at 53.34 95.25 0)
-      (effects (font (size 1.27 1.27)) hide)
-    )
-    (property "Value" "VBUS" (at 53.34 87.7316 0)
-      (effects (font (size 1.27 1.27)))
-    )
-    (property "Footprint" "" (at 53.34 91.44 0)
-      (effects (font (size 1.27 1.27)) hide)
-    )
-    (property "Datasheet" "" (at 53.34 91.44 0)
-      (effects (font (size 1.27 1.27)) hide)
-    )
-    (property "Mfr." "" (at 53.34 91.44 0)
-      (effects (font (size 1.27 1.27)) hide)
-    )
-    (property "Mfr. No." "" (at 53.34 91.44 0)
-      (effects (font (size 1.27 1.27)) hide)
-    )
-    (property "Distributor" "" (at 53.34 91.44 0)
-      (effects (font (size 1.27 1.27)) hide)
-    )
-    (property "Order Number" "" (at 53.34 91.44 0)
+  (symbol (lib_id "power:VBUS") (at 53.34 97.79 0) (mirror y) (unit 1)
+    (in_bom yes) (on_board yes) (dnp no)
+    (property "Reference" "#PWR08" (at 53.34 101.6 0)
+      (effects (font (size 1.27 1.27)) hide)
+    )
+    (property "Value" "VBUS" (at 53.34 94.0816 0)
+      (effects (font (size 1.27 1.27)))
+    )
+    (property "Footprint" "" (at 53.34 97.79 0)
+      (effects (font (size 1.27 1.27)) hide)
+    )
+    (property "Datasheet" "" (at 53.34 97.79 0)
+      (effects (font (size 1.27 1.27)) hide)
+    )
+    (property "Mfr." "" (at 53.34 97.79 0)
+      (effects (font (size 1.27 1.27)) hide)
+    )
+    (property "Mfr. No." "" (at 53.34 97.79 0)
+      (effects (font (size 1.27 1.27)) hide)
+    )
+    (property "Distributor" "" (at 53.34 97.79 0)
+      (effects (font (size 1.27 1.27)) hide)
+    )
+    (property "Order Number" "" (at 53.34 97.79 0)
       (effects (font (size 1.27 1.27)) hide)
     )
@@
     )
   )
-  (symbol (lib_id "Switch:SW_DIP_x04") (at 123.19 71.12 0) (unit 1)
+  (symbol (lib_id "Switch:SW_DIP_x01") (at 123.19 71.12 0) (unit 1)
     (in_bom yes) (on_board yes) (dnp no) (fields_autoplaced)
     (property "Reference" "SW1" (at 123.19 59.69 0)
@@
       (effects (font (size 1.27 1.27)) hide)
     )
-    (property "Datasheet" "https://www.mouser.de/datasheet/2/418/8/ENG_CD_1825058_T-687817.pdf" (at 123.19 71.12 0)
+    (property "Datasheet" "~" (at 123.19 71.12 0)
       (effects (font (size 1.27 1.27)) hide)
     )
@@
     (pin "1")
     (pin "2")
-    (pin "3")
-    (pin "4")
-    (pin "5")
-    (pin "6")
-    (pin "7")
-    (pin "8")
-    (instances
-      (project "ZSWatch-Dock"
+    (instances
+      (project "ZSWatch-Dock"

Commit message: - Add QR code with link to GitHub repository - Add switch to enable / disable charging - Remove reset line from STM32 to the watch connector
Signed-off-by: Daniel Kampert <DanielKampert@kampis-elektroecke.de>
Parts:
- removed SW1: CONFIG, Button_Switch_SMD:SW_DIP_SPSTx04_Slide_Omron_A6S-410x_W8.9mm_P2.54mm, symbol Switch:SW_DIP_x01
- removed X2: GPIO, Connector_PinHeader_2.54mm:PinHeader_1x01_P2.54mm_Vertical, symbol Connector_Generic:Conn_01x01
- added D3: DEBUG, LED_SMD:LED_0603_1608Metric, symbol Device:LED
- added Q1: BSH205G2AR, Package_TO_SOT_SMD:SOT-23, symbol Nexperia:BSH205G2AR
- added R10: 220R, Resistor_SMD:R_0603_1608Metric, symbol Device:R_Small
- added R9: 100k, Resistor_SMD:R_0603_1608Metric, symbol Device:R_Small
- SW2: footprint Button_Switch_SMD:SW_DIP_SPSTx01_Slide_6.7x4.1mm_W6.73mm_P2.54mm_LowProfile_JPin -> Button_Switch_SMD:SW_SP3T_PCM13; symbol Switch:SW_DIP_x01 -> Switch:SW_DPST; Distributor (none) -> Mouser; Mfr. (none) -> C&K; Mfr. No. (none) -> PCM13SMTR; Order Number (none) -> 611-PCM13SMTR
Connections:
- net ZSWatch_RESETn is gone; now on net GND: X1.3 (Pin_3)
- net +3V3: now also D3.2 (A)
- net GND: now also SW2.1, SW2.3
- net SWDRESETn: no longer IC3.10 (B1), IC4.11 (PA1)
- net VBUS: now also Q1.2 (S), R9.2; no longer SW2.2
- net at X1.5 (Pin_5): now also Q1.3 (D); no longer SW2.1
- net STM32_RxD: no longer names the net of IC4.31 (PA10)
- net STM32_SWD_RESETn: no longer names the net of IC3.2 (A1)
- net STM32_TxD: no longer names the net of IC4.30 (PA9)
- new net: Q1.1 (G), R9.1, SW2.4
- new net: D3.1 (K), R10.1
- new net CHARGE: R10.2, SW2.2
- no-connect marks 33 -> 38
Other:
- note added: "LEDs"
- note added: "NOTE: The watch PCB is configured for USB per default. and the signal must be pulled to GND to switch to SWD. The logic is compatible with the watch hardware 3 and below, since the switch can be used as a normal reset signal."
- note removed: "Debug LED"
- note removed: "Status LED"
- note removed: "ZSWatch Reset Config"
- moved on the sheet: D1, D2, R1, R2, X1, X3

Commit message: fixup! - Add QR code with link to GitHub repository - Add switch to enable / disable charging - Remove reset line from STM32 to the watch connector
Other:
- note added: "NOTE: The watch PCB is configured for USB per default. and the signal must be pulled to GND to switch to SWD."
- note removed: "NOTE: The watch PCB is configured for USB per default. and the signal must be pulled to GND to switch to SWD. The logic is compatible with the watch hardware 3 and below, since the switch can be used as a normal reset signal."
- moved on the sheet: Q1, R9, SW2, X1

Commit message: - Fix wrong part number for inductor
Parts:
- removed R6: 0R, Resistor_SMD:R_0603_1608Metric, symbol Device:R_Small
- C10, C11, C8, C9, IC4: Config (none) -> +INT_JLINK,-EXT_JLINK
- L1: Mfr. TAIYO YUDEN -> TDK; Mfr. No. LSCNB1608HKT1R0MD -> MLZ1608N100LT000; Order Number 963-LSCNB1608HKT1R0MD -> 810-MLZ1608N100LT000
- R4, R5: Config (none) -> -INT_JLINK,+EXT_JLINK
Other:
- note added: "NOTE: The watch PCB is configured for USB per default. Thus the USB / SWD signal must be pulled to GND to use SWD."
- note removed: "NOTE: The watch PCB is configured for USB per default. and the signal must be pulled to GND to switch to SWD."

Commit message: Add KiBot workflow
Parts:
- added JP1: SEL, Jumper:SolderJumper-3_P1.3mm_Bridged12_Pad1.0x1.5mm_NumberLabels, symbol Jumper:Jumper_3_Bridged12
- C10, C11, C8, C9, IC4: CONFIG (none) -> +INT_JLINK; Config +INT_JLINK,-EXT_JLINK -> (none)
- C5, C7, IC3: CONFIG (none) -> +INT_JLINK
- R4, R5: CONFIG (none) -> +EXT_JLINK; Config -INT_JLINK,+EXT_JLINK -> (none); now fitted; now in the parts list
Connections:
- net +3V3: now also JP1.3 (B)
- net GND: now also JP1.1 (A); no longer X1.3 (Pin_3)
- new net: JP1.2 (C), X1.3 (Pin_3)
Other:
- moved on the sheet: X1
