File: project/ZSWatch-Dock.kicad_sch (KiCad schematic)
At the start: 34 parts, among them IC1 XC9265C181MR-G, IC2 MIC5219-3.3YM5, IC3 NTS0104GU12, IC4 STM32F072CBT6, Q1 BSH205G2AR, SW2 CHARGE, X1 WATCH, X3 DEBUG, X4 USB4105-GF-A

Commit message: Fix wrong KiBot variant names
Parts:
- C10, C11, C5, C7, C8, C9, IC3, IC4: CONFIG +INT_JLINK -> +INT
- R4, R5: CONFIG +EXT_JLINK -> +EXT
Changed lines of the file:
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@@
       (effects (font (size 1.27 1.27)) hide)
     )
-    (property "CONFIG" "+INT_JLINK" (at 186.69 45.72 0)
+    (property "CONFIG" "+INT" (at 186.69 45.72 0)
       (effects (font (size 1.27 1.27)) hide)
     )
@@
       (effects (font (size 1.27 1.27)) hide)
     )
-    (property "CONFIG" "+EXT_JLINK" (at 144.78 29.21 0)
+    (property "CONFIG" "+EXT" (at 144.78 29.21 0)
       (effects (font (size 1.27 1.27)) hide)
     )
@@
       (effects (font (size 1.27 1.27)) hide)
     )
-    (property "CONFIG" "+INT_JLINK" (at 199.39 66.04 0)
+    (property "CONFIG" "+INT" (at 199.39 66.04 0)
       (effects (font (size 1.27 1.27)) hide)
     )
@@
       (effects (font (size 1.27 1.27)) hide)
     )
-    (property "CONFIG" "+INT_JLINK" (at 121.92 110.49 0)
+    (property "CONFIG" "+INT" (at 121.92 110.49 0)
       (effects (font (size 1.27 1.27)) hide)
     )
@@
       (effects (font (size 1.27 1.27)) hide)
     )
-    (property "CONFIG" "+INT_JLINK" (at 190.5 116.84 0)
+    (property "CONFIG" "+INT" (at 190.5 116.84 0)
       (effects (font (size 1.27 1.27)) hide)
     )
@@
       (effects (font (size 1.27 1.27)) hide)
     )
-    (property "CONFIG" "+INT_JLINK" (at 127 91.44 0)
+    (property "CONFIG" "+INT" (at 127 91.44 0)
       (effects (font (size 1.27 1.27)) hide)
     )
@@
       (effects (font (size 1.27 1.27)) hide)
     )
-    (property "CONFIG" "+INT_JLINK" (at 118.11 91.44 0)
+    (property "CONFIG" "+INT" (at 118.11 91.44 0)
       (effects (font (size 1.27 1.27)) hide)
     )
@@
       (effects (font (size 1.27 1.27)) hide)
     )
-    (property "CONFIG" "+INT_JLINK" (at 184.15 66.04 0)
+    (property "CONFIG" "+INT" (at 184.15 66.04 0)
       (effects (font (size 1.27 1.27)) hide)
     )
@@
       (effects (font (size 1.27 1.27)) hide)
     )
-    (property "CONFIG" "+EXT_JLINK" (at 144.78 38.1 0)
+    (property "CONFIG" "+EXT" (at 144.78 38.1 0)
       (effects (font (size 1.27 1.27)) hide)
     )
@@
       (effects (font (size 1.27 1.27)) hide)
     )
-    (property "CONFIG" "+INT_JLINK" (at 196.85 45.72 0)
-      (effects (font (size 1.27 1.27)) hide)
-    )
+    (property "CONFIG" "+INT" (at 196.85 45.72 0)
+      (effects (font (size 1.27 1.27)) hide)
+    )

Commit message: Add second USB interface, rename variants
Parts:
- removed JP1: SEL, Jumper:SolderJumper-3_P1.3mm_Bridged12_Pad1.0x1.5mm_NumberLabels, symbol Jumper:Jumper_3_Bridged12
- added C3: 100n, Capacitor_SMD:C_0603_1608Metric, symbol Device:C_Small
- added IC2: TS3USB221A, Package_QFN:UQFN-10_1.55x2.05mm_P0.5mm, symbol TexasInstruments_Kampi:TS3USB221A
- added R1, R3: 100k, Resistor_SMD:R_0603_1608Metric, symbol Device:R_Small
- added R14, R15: 5k1, Resistor_SMD:R_0603_1608Metric, symbol Device:R_Small
- added R4, R5: 0R, Resistor_SMD:R_0603_1608Metric, symbol Device:R_Small
- added SW2: SEL, Button_Switch_SMD:SW_SPDT_PCM12, symbol Switch:SW_DPDT_x2
- added X4: DATA, Connector_USB:USB_C_Receptacle_GCT_USB4105-xx-A_16P_TopMnt_Horizontal, symbol Connector:USB_C_Receptacle_USB2.0
- C10: renamed from C9; CONFIG +INT -> +FULL
- C11: renamed from C10; CONFIG +INT -> +FULL
- C12: renamed from C11; CONFIG +INT -> +FULL
- C6: renamed from C5; CONFIG +INT -> +FULL
- C8: renamed from C7; CONFIG +INT -> +FULL
- C9: renamed from C8; CONFIG +INT -> +FULL
- IC4: renamed from IC3; CONFIG +INT -> +FULL
- IC5: renamed from IC4; CONFIG +INT -> +FULL
- R7: renamed from R4; CONFIG +EXT -> +REDUCED,+MINIMUM
- R8: renamed from R5; CONFIG +EXT -> +REDUCED,+MINIMUM
- SW1: renamed from SW2; footprint Button_Switch_SMD:SW_SP3T_PCM13 -> Button_Switch_SMD:SW_SPDT_PCM12; symbol Switch:SW_DPST -> Switch:SW_DPDT_x2; Mfr. No. PCM13SMTR -> PCM12SMTR; Order Number 611-PCM13SMTR -> 611-PCM12SMTR
- X3: renamed from X4; value USB4105-GF-A -> DEBUG
- renumbered C3 to C4, C4 to C5, C6 to C7, IC2 to IC3, R2 to R10, R10 to R11, R7 to R12, R8 to R13, R9 to R2, R3 to R6, R1 to R9, X3 to X2
Connections:
- net +3V3: now also C3.1, IC2.10 (VDD), R1.1
- net CHARGE: now also Q1.1 (G), R2.1, SW1.3 (C); no longer SW1.2
- net GND: now also SW1.2 (B), C3.2, IC2.5 (GND), R14.2, R15.1, R3.2, SW2.2 (B), X4.A1 (GND), X4.A12 (GND), X4.B1 (GND), X4.B12 (GND), X4.S1 (SHIELD); no longer SW1.1, SW1.3
- net VBUS: now also X4.A4 (VBUS), X4.A9 (VBUS), X4.B4 (VBUS), X4.B9 (VBUS)
- net SEL_SWD: now reaches X1.3 (Pin_3)
- net SEL_SWD: now also IC2.9 (S), R1.2, SW2.3 (C)
- net USB_DATA_N renamed USB1_DATA_N
- net USB_DATA_P renamed USB1_DATA_P
- net ZSWatch_SWDCLK renamed D+/SWDCLK
- net D+/SWDCLK: now also IC2.8 (D+), R5.2; no longer IC4.4 (A3)
- net ZSWatch_SWDIO renamed D-/SWDIO
- net D-/SWDIO: now also IC2.7 (D-), R4.2; no longer IC4.5 (A4)
- new net: IC2.6 (~{OE}), R3.1
- new net: R15.2, X4.B5 (CC2)
- new net: R14.1, X4.A5 (CC1)
- new net SWDCLK_WATCH: IC2.3 (2D+), IC4.4 (A3), R5.1
- new net SWDIO_WATCH: IC2.4 (2D-), IC4.5 (A4), R4.1
- new net USB2_DATA_N: IC2.2 (1D-), X4.A7 (D-), X4.B7 (D-)
- new net USB2_DATA_P: IC2.1 (1D+), X4.A6 (D+), X4.B6 (D+)
- no-connect marks 38 -> 40
Other:
- note added: "NOTE: The SWD bridge is needed when the USB option isn´t selected."
- note added: "S Channel Function L HSD1+ and HSD1- USB H HSD2+ and HSD2- SWD (Default)"
- note added: "USB / SWD Switch"
- note removed: "NOTE: The watch PCB is configured for USB per default. Thus the USB / SWD signal must be pulled to GND to use SWD."
- moved on the sheet: C1, C2, C4, C5, C7, D1, D2, D3, IC1, IC3, L1, Q1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

Commit message: - Remove old documentation - Increase drill hole size for watch connector to 1.4 mm - Add mounting holes for a zipper as cable protection - Move mounting holes to a new position into the corners - Set origin for step export in KiBot configuration
Connections:
- no-connect marks 40 -> 42
Other:
- note added: "NOTE: Change the hole size of the watch connector to 1.4 mm"
- moved on the sheet: C10, C11, C12, C3, C6, C8, C9, IC4, IC5, R4, R5, R6

Commit message: Remove 3V3 regulator in minimal variant
Parts:
- C4, C5, C7, IC3: CONFIG (none) -> +FULL,+REDUCED
Changed lines of the file:
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@@
+      (effects (font (size 1.27 1.27)) hide)
+    )
+    (property "CONFIG" "+FULL,+REDUCED" (at 119.38 36.83 0)
       (effects (font (size 1.27 1.27)) hide)
     )
@@
     )
     (property "Order Number" "998-MIC5219-3.3YM5TR" (at 86.36 31.75 0)
+      (effects (font (size 1.27 1.27)) hide)
+    )
+    (property "CONFIG" "+FULL,+REDUCED" (at 86.36 31.75 0)
       (effects (font (size 1.27 1.27)) hide)
     )
@@
       (effects (font (size 1.27 1.27)) hide)
     )
+    (property "CONFIG" "+FULL,+REDUCED" (at 109.22 36.83 0)
+      (effects (font (size 1.27 1.27)) hide)
+    )
     (pin "1")
     (pin "2")
@@
       (effects (font (size 1.27 1.27)) hide)
     )
+    (property "CONFIG" "+FULL,+REDUCED" (at 99.06 36.83 0)
+      (effects (font (size 1.27 1.27)) hide)
+    )

Commit message: Add jumper to select the right voltage for VTarget on STM32 SWD
Parts:
- added R1, R3: 0R, Resistor_SMD:R_0603_1608Metric, symbol Device:R_Small
- renumbered C7 to C6, C6 to C7, R6 to R10, R9 to R11, R10 to R12, R11 to R13, R12 to R14, R13 to R15, R14 to R16, R15 to R17, R1 to R2, R2 to R4, R3 to R5, R4 to R6, R5 to R7, R7 to R8, R8 to R9, SW2 to SW1, SW1 to SW2
Connections:
- net +1V8: now also R3.1
- net +3V3: now also R1.2; no longer X2.1 (VTref)
- new net: R1.1, R3.2, X2.1 (VTref)

Commit message: Remove watch connector from BOM and from 3D data
Parts:
- X1: now left out of the parts list
Changed lines of the file:
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@@
   )
   (symbol (lib_id "Connector_Generic:Conn_01x05") (at 22.86 67.31 0) (mirror y) (unit 1)
-    (in_bom yes) (on_board yes) (dnp no)
+    (in_bom no) (on_board yes) (dnp no)
     (property "Reference" "X1" (at 20.32 66.675 0)
       (effects (font (size 1.27 1.27)) (justify left))
@@
       (effects (font (size 1.27 1.27)) hide)
     )
+    (property "CONFIG" "" (at 22.86 67.31 0)
+      (effects (font (size 1.27 1.27)) hide)
+    )
