File: project/ZSWatch-Dock.kicad_sch (KiCad schematic)
At the start: 45 parts, among them IC1 XC9265C181MR-G, IC2 TS3USB221A, IC3 MIC5219-3.3YM5, IC4 NTS0104GU12, IC5 STM32F072CBT6, Q1 BSH205G2AR, SW1 SEL, SW2 CHARGE, X1 WATCH, X2 DEBUG, X3 DEBUG, X4 DATA

Commit message: Add note for setting SEL to high per default to support rev <5
Other:
- note added: "NOTE: SEL must be high in default mode because in revisions <5 SEL is used as MCU reset."
Changed lines of the file:
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@@
     (effects (font (size 3 3)) (justify left bottom))
+  )
+  (text "NOTE:\nSEL must be high in default mode\nbecause in revisions <5 SEL is used\nas MCU reset."
+    (at 13.97 223.52 0)
+    (effects (font (size 1.27 1.27)) (justify left bottom))
   )
   (text "1V8 Regulator" (at 13.97 17.78 0)

Commit message: Add debounce capacitor to SEL-Switch
Parts:
- added C2: 100n, Capacitor_SMD:C_0603_1608Metric, symbol Device:C_Small
- added R3: 1k, Resistor_SMD:R_0603_1608Metric, symbol Device:R_Small
- renumbered C9 to C10, C10 to C11, C11 to C12, C12 to C13, C2 to C3, C3 to C4, C4 to C5, C5 to C6, C6 to C7, C7 to C8, C8 to C9, R9 to R10, R10 to R11, R11 to R12, R12 to R13, R13 to R14, R14 to R15, R15 to R16, R16 to R17, R17 to R18, R3 to R2, R2 to R4, R4 to R5, R5 to R6, R6 to R7, R7 to R8, R8 to R9
Connections:
- net GND: now also C2.2
- net SEL_SWD: now also C2.1, R3.1; no longer SW1.3 (C)
- new net: R3.2, SW1.3 (C)
Other:
- moved on the sheet: C4, IC2, R4, R6, R7, R8, SW1A

Commit message: Change power supply for CHARGE LED to VBUS
Parts:
- D3: value DEBUG -> CHARGE
Connections:
- net +3V3: no longer D3.2 (A)
- net VBUS: now also D3.2 (A)
Changed lines of the file:
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@@
-    )
-  )
-  (symbol (lib_id "power:+3V3") (at 373.38 246.38 0) (unit 1)
-    (in_bom yes) (on_board yes) (dnp no) (fields_autoplaced)
-    (property "Reference" "#PWR048" (at 373.38 250.19 0)
-      (effects (font (size 1.27 1.27)) hide)
-    )
-    (property "Value" "+3V3" (at 373.38 242.57 0)
-      (effects (font (size 1.27 1.27)))
-    )
-    (property "Footprint" "" (at 373.38 246.38 0)
-      (effects (font (size 1.27 1.27)) hide)
-    )
-    (property "Datasheet" "" (at 373.38 246.38 0)
-      (effects (font (size 1.27 1.27)) hide)
-    )
-    (pin "1")
-    (instances
-      (project "ZSWatch-Dock"
-        (path "/74a2d9cd-6788-49ca-9d1d-a5e7b3102f3e"
-          (reference "#PWR048") (unit 1)
-        )
-      )
     )
   )
@@
       (effects (font (size 1.27 1.27)))
     )
-    (property "Value" "DEBUG" (at 382.5875 242.57 0)
+    (property "Value" "CHARGE" (at 382.5875 242.57 0)
       (effects (font (size 1.27 1.27)))
     )
@@
     )
     (property "Order Number" "710-150060VS75003" (at 381 247.65 0)
+      (effects (font (size 1.27 1.27)) hide)
+    )
+    (property "CONFIG" "" (at 381 247.65 0)
       (effects (font (size 1.27 1.27)) hide)
     )
@@
         )
       )
+    )
+  )
+  (symbol (lib_id "power:VBUS") (at 373.38 246.38 0) (mirror y) (unit 1)
+    (in_bom yes) (on_board yes) (dnp no)
+    (property "Reference" "#PWR048" (at 373.38 250.19 0)
+      (effects (font (size 1.27 1.27)) hide)
+    )
+    (property "Value" "VBUS" (at 373.38 242.6716 0)
+      (effects (font (size 1.27 1.27)))
+    )
+    (property "Footprint" "" (at 373.38 246.38 0)
+      (effects (font (size 1.27 1.27)) hide)
+    )
+    (property "Datasheet" "" (at 373.38 246.38 0)
+      (effects (font (size 1.27 1.27)) hide)
+    )
+    (property "Mfr." "" (at 373.38 246.38 0)
+      (effects (font (size 1.27 1.27)) hide)
+    )
+    (property "Mfr. No." "" (at 373.38 246.38 0)
+      (effects (font (size 1.27 1.27)) hide)
+    )
+    (property "Distributor" "" (at 373.38 246.38 0)
+      (effects (font (size 1.27 1.27)) hide)
+    )
+    (property "Order Number" "" (at 373.38 246.38 0)
+      (effects (font (size 1.27 1.27)) hide)
+    )
+    (pin "1")
+    (instances
+      (project "ZSWatch-Dock"
+        (path "/74a2d9cd-6788-49ca-9d1d-a5e7b3102f3e"
+          (reference "#PWR048") (unit 1)
+        )
+      )

Commit message: Remove STATUS LED in minimal variant
Parts:
- D1, R12: CONFIG (none) -> +FULL,+REDUCED
Changed lines of the file:
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@@
+      (effects (font (size 1.27 1.27)) hide)
+    )
+    (property "CONFIG" "+FULL,+REDUCED" (at 391.16 224.79 0)
       (effects (font (size 1.27 1.27)) hide)
     )
@@
       (effects (font (size 1.27 1.27)) hide)
     )
+    (property "CONFIG" "+FULL,+REDUCED" (at 381 224.79 0)
+      (effects (font (size 1.27 1.27)) hide)
+    )

Commit message: Add debounce capacitor for SEL pin to reduced variant, remove STATUS LED in reduced variant
Parts:
- C2: CONFIG +FULL -> +FULL,+REDUCED
- D1, R12: CONFIG +FULL,+REDUCED -> +FULL
Changed lines of the file:
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@@
       (effects (font (size 1.27 1.27)) hide)
     )
-    (property "CONFIG" "+FULL" (at 45.72 270.51 0)
+    (property "CONFIG" "+FULL,+REDUCED" (at 45.72 270.51 0)
       (effects (font (size 1.27 1.27)) hide)
     )
@@
       (effects (font (size 1.27 1.27)) hide)
     )
-    (property "CONFIG" "+FULL,+REDUCED" (at 391.16 224.79 0)
+    (property "CONFIG" "+FULL" (at 391.16 224.79 0)
       (effects (font (size 1.27 1.27)) hide)
     )
@@
       (effects (font (size 1.27 1.27)) hide)
     )
-    (property "CONFIG" "+FULL,+REDUCED" (at 381 224.79 0)
-      (effects (font (size 1.27 1.27)) hide)
-    )
+    (property "CONFIG" "+FULL" (at 381 224.79 0)
+      (effects (font (size 1.27 1.27)) hide)
+    )

Commit message: - Replace QR code with area for QR code - Add isolation diode to disconnect both VBUS from each other - Add new logo
Signed-off-by: Daniel Kampert <DanielKampert@kampis-elektroecke.de>
Parts:
- added D103: BAT64-05, Package_TO_SOT_SMD:SOT-23-3, symbol Device:D_Schottky_Dual_CommonCathode_AAK_Parallel
- R5: Mfr. No. RT0603FRE07100KL -> RC0603FR-07100KL; Order Number 603-RT0603FRE07100KL -> 603-RC0603FR-07100KL
Connections:
- net VBUS: now also D103.3 (A); no longer X3.A4 (VBUS), X3.A9 (VBUS), X3.B4 (VBUS), X3.B9 (VBUS), X4.A4 (VBUS), X4.A9 (VBUS), X4.B4 (VBUS), X4.B9 (VBUS)
- new net: D103.1 (K), X4.A4 (VBUS), X4.A9 (VBUS), X4.B4 (VBUS), X4.B9 (VBUS)
- new net: D103.2 (K), X3.A4 (VBUS), X3.A9 (VBUS), X3.B4 (VBUS), X3.B9 (VBUS)
Other:
- moved on the sheet: R15, R16, R17, R18, X3, X4

Commit message: Initialize branch for rev 4, add connector for current measurement of the watch
Parts:
- added R103: 0R, Resistor_SMD:R_0805_2012Metric_Pad1.20x1.40mm_HandSolder, symbol Device:R_Small
- added X103: Current, Connector_PinHeader_2.54mm:PinHeader_1x02_P2.54mm_Horizontal, symbol Connector_Generic:Conn_01x02
- renumbered C1 to C101, C2 to C102, C3 to C103, C4 to C104, C5 to C105, C6 to C106, C7 to C107, C8 to C108, C9 to C109, C10 to C110, C11 to C111, C12 to C112, C13 to C113, D1 to D101, D2 to D102, D3 to D103, D103 to D104, IC1 to IC101, IC2 to IC102, IC3 to IC103, IC4 to IC104, IC5 to IC105, L1 to L101, Q1 to Q101, R1 to R101, R2 to R102, R3 to R104, R4 to R105, R5 to R106, R6 to R107, R7 to R108, R8 to R109, R9 to R110, R10 to R111, R11 to R112, R15 to R113, R16 to R114, R17 to R115, R18 to R116, R12 to R117, R13 to R118, R14 to R119, SW1 to SW101, SW2 to SW102, X1 to X101, X2 to X102, X3 to X104, X4 to X105
Connections:
- net at X101.5 (Pin_5): now also R103.2, X103.2 (Pin_2); no longer Q101.3 (D)
- new net: Q101.3 (D), R103.1, X103.1 (Pin_1)
Other:
- moved on the sheet: Q101, R106, SW102A, X101

Commit message: Replace protection diodes for VBUS with LM66200
Parts:
- removed D104: BAT64-05, Package_TO_SOT_SMD:SOT-23-3, symbol Device:D_Schottky_Dual_CommonCathode_AAK_Parallel
- added IC106: LM66200, Package_SOT_SMD:SOT-5X3-8, symbol Texas Instruments:LM66200
Connections:
- net GND: now also IC106.1 (GND), IC106.4 (~{ON}), IC106.5 (GND)
- net VBUS: now also IC106.2 (VOUT), IC106.7 (VOUT)
- net at X105.A4 (VBUS), X105.A9 (VBUS), X105.B4 (VBUS)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: now also IC106.6 (VIN2)
- net at X104.A4 (VBUS), X104.A9 (VBUS), X104.B4 (VBUS)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: now also IC106.3 (VIN1)
- no-connect marks 42 -> 43
Other:
- moved on the sheet: R113, R114, R115, R116, X104, X105
